Commit message: update robot material

File: src/my_robot/urdf/my_robot.xacro (robot description, xacro)
@@ -185,14 +185,17 @@
   </joint>
   <gazebo reference="chassis">
-    <material>Gazebo/Blue</material>
+    <material>Gazebo/Indigo</material>
   </gazebo>
   <gazebo reference="left_wheel">
-    <material>Gazebo/Green</material>
+    <material>Gazebo/Turquoise</material>
   </gazebo>
   <gazebo reference="right_wheel">
-    <material>Gazebo/Green</material>
+    <material>Gazebo/Turquoise</material>
   </gazebo>
   <gazebo reference="camera">
-    <material>Gazebo/Yellow</material>
+    <material>Gazebo/RedGlow</material>
+  </gazebo>
+  <gazebo reference="hokuyo">
+    <material>Gazebo/DarkMagentaTransparent</material>
   </gazebo>
 </robot>

Commit message: adding database

File: src/my_robot/urdf/my_robot.xacro (robot description, xacro)
@@ -152,4 +152,11 @@
     <dynamics damping="1.0" friction="1.0"/>
   </joint>
+  <link name="camera_link_optical">
+  </link>
+  <joint name="camera_optical_joint" type="fixed">
+    <origin xyz="0 0 0" rpy="-1.5707 0 -1.5707"/>
+    <parent link="camera"/>
+    <child link="camera_link_optical"/>
+  </joint>
   <link name='hokuyo'>
     <pose>0 0 0 0 0 0</pose>
